File: CP2_Compensacion/Regulador Lineal.kicad_sch (KiCad schematic)
At the start: 22 parts, among them Q1 BD140, Q10 BD139, Q2 BD140, Q3 BD139, Q4 BD139, Q5 TIP42C, Q6 BD139, Q7 BD139, Q8 BD139

Commit message: Add files via upload
Parts:
- removed C3: 1u, Capacitor_SMD:CP_Elec_6.3x5.7, symbol Device:C
- removed RL1: 10, Resistor_THT:R_Axial_DIN0204_L3.6mm_D1.6mm_P5.08mm_Horizontal, symbol Device:R
- removed Vin1: 9.5, Connector_PinHeader_1.00mm:PinHeader_1x01_P1.00mm_Horizontal, symbol Device:Battery_Cell
- removed Vref1: 2.5, Connector_PinHeader_1.00mm:PinHeader_1x01_P1.00mm_Horizontal, symbol Device:Battery_Cell
- added J1, J2: conn_vreg, Connector_PinHeader_1.00mm:PinHeader_1x01_P1.00mm_Vertical, symbol Connector:Conn_01x01_Pin
- added J3: conn_rl_gnd, Connector_PinHeader_1.00mm:PinHeader_1x01_P1.00mm_Vertical, symbol Connector:Conn_01x01_Pin
- added J4: conn_rl, Connector_PinHeader_1.00mm:PinHeader_1x01_P1.00mm_Vertical, symbol Connector:Conn_01x01_Pin
- added R3: 470, Resistor_THT:R_Axial_DIN0204_L3.6mm_D1.6mm_P5.08mm_Horizontal, symbol Device:R
- added U1: TL431LP, Package_TO_SOT_THT:TO-92_Inline, symbol Reference_Voltage:TL431LP
Connections:
- net GND: now also J1.1 (Pin_1), J3.1 (Pin_1), U1.2 (A)
- net at Q5.3 (E), R8.1, R9.1: now also J2.1 (Pin_1), R3.1
- net at Q3.3 (B), R1.1: now also R3.2, U1.1 (REF), U1.3 (K)
- net at Q7.1 (E), R4.2, R5.1: now also J4.1 (Pin_1)

Commit message: Add files via upload
Parts:
- removed J1, J2: conn_vreg, Connector_PinHeader_1.00mm:PinHeader_1x01_P1.00mm_Vertical, symbol Connector:Conn_01x01_Pin
- removed J3: conn_rl_gnd, Connector_PinHeader_1.00mm:PinHeader_1x01_P1.00mm_Vertical, symbol Connector:Conn_01x01_Pin
- added J1: I1, Connector_PinHeader_2.54mm:PinHeader_1x02_P2.54mm_Vertical, symbol Connector:Conn_01x02_Pin
- added J2: I2, Connector_PinHeader_2.54mm:PinHeader_1x02_P2.54mm_Vertical, symbol Connector:Conn_01x02_Pin
- added J3: I3, Connector_PinHeader_2.54mm:PinHeader_1x02_P2.54mm_Vertical, symbol Connector:Conn_01x02_Pin
- added J5: out, TerminalBlock_Phoenix:TerminalBlock_Phoenix_MKDS-1,5-2-5.08_1x02_P5.08mm_Horizontal, symbol Connector:Screw_Terminal_01x02
- added J6: V1, Connector_PinHeader_2.54mm:PinHeader_1x01_P2.54mm_Vertical, symbol Connector:Conn_01x01_Pin
- added J7: in, TerminalBlock_Phoenix:TerminalBlock_Phoenix_MKDS-1,5-2-5.08_1x02_P5.08mm_Horizontal, symbol Connector:Screw_Terminal_01x02
- C4: footprint Capacitor_SMD:CP_Elec_6.3x4.5 -> Capacitor_THT:C_Disc_D4.3mm_W1.9mm_P5.00mm
- J4: value conn_rl -> gnd; footprint Connector_PinHeader_1.00mm:PinHeader_1x01_P1.00mm_Vertical -> Connector_PinHeader_2.54mm:PinHeader_1x01_P2.54mm_Vertical
Connections:
- net GND: now also J4.1 (Pin_1), J5.1 (Pin_1), J7.1 (Pin_1)
- net at Q5.2 (C), Q6.1 (E): now also J1.2 (Pin_2); no longer R4.1, R7.1
- net at Q5.3 (E), R3.1, R8.1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: now also J7.2 (Pin_2)
- net at Q3.1 (E), Q4.1 (E): now also J2.1 (Pin_1); no longer Q8.2 (C)
- net at Q3.3 (B), R1.1, R3.2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: now also J6.1 (Pin_1)
- net at Q7.1 (E), R4.2, R5.1: now also J5.2 (Pin_2); no longer J4.1 (Pin_1)
- net at R5.2, R6.1: now also J3.1 (Pin_1); no longer Q4.3 (B)
- new net: J3.2 (Pin_2), Q4.3 (B)
- new net: J1.1 (Pin_1), R4.1, R7.1
- new net: J2.2 (Pin_2), Q8.2 (C)

Commit message: Correcion del esquematico KiCad
Connections:
- net at Q1.3 (B), Q2.3 (B), Q3.2 (C): now also Q1.2 (C); no longer Q1.1 (E)
- net at C4.2, Q4.2 (C), Q6.3 (B)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: now also Q2.2 (C); no longer Q2.1 (E)
- net at R8.2: now also Q1.1 (E); no longer Q1.2 (C)
- net at R9.2: now also Q2.1 (E); no longer Q2.2 (C)
Other:
- moved on the sheet: Q1
