File: CP2_Compensacion/Regulador Lineal.kicad_pcb (KiCad board)
At the start: 2 copper layers, 64 x 51 mm, 27 parts, among them J1 I1, J2 I2, J3 I3, J4 gnd, J5 out, J6 V1, J7 in, Q1 BD140, Q10 BD139, Q2 BD140, Q3 BD139, Q4 BD139, Q5 TIP42C, Q6 BD139, Q7 BD139, Q8 BD139, U1 TL431LP

Commit message: PCB ok
Parts:
- added C4: 330n, Capacitor_THT:C_Rect_L7.0mm_W2.0mm_P5.00mm, F.Cu at (150.1, 137.8)
- added C4: 330n, Capacitor_THT:C_Rect_L7.0mm_W2.0mm_P5.00mm, F.Cu at (233.9, 137.8)
- added C4: 330n, Capacitor_THT:C_Rect_L7.0mm_W2.0mm_P5.00mm, F.Cu at (233.9, 66.6)
- added C4: 330n, Capacitor_THT:C_Rect_L7.0mm_W2.0mm_P5.00mm, F.Cu at (68.8, 66.7)
- added C4: 330n, Capacitor_THT:C_Rect_L7.0mm_W2.0mm_P5.00mm, F.Cu at (68.8, 137.8)
- added J1: I1, Connector_PinHeader_2.54mm:PinHeader_1x02_P2.54mm_Vertical, F.Cu at (172.1, 127.4)
- added J1: I1, Connector_PinHeader_2.54mm:PinHeader_1x02_P2.54mm_Vertical, F.Cu at (90.9, 56.3)
- added J1: I1, Connector_PinHeader_2.54mm:PinHeader_1x02_P2.54mm_Vertical, F.Cu at (256.0, 56.3)
- added J1: I1, Connector_PinHeader_2.54mm:PinHeader_1x02_P2.54mm_Vertical, F.Cu at (90.9, 127.4)
- added J1: I1, Connector_PinHeader_2.54mm:PinHeader_1x02_P2.54mm_Vertical, F.Cu at (256.0, 127.4)
- added J2: I2, Connector_PinHeader_2.54mm:PinHeader_1x02_P2.54mm_Vertical, F.Cu at (56.7, 155.5)
- added J2: I2, Connector_PinHeader_2.54mm:PinHeader_1x02_P2.54mm_Vertical, F.Cu at (221.8, 84.4)
- added J2: I2, Connector_PinHeader_2.54mm:PinHeader_1x02_P2.54mm_Vertical, F.Cu at (137.9, 155.5)
- added J2: I2, Connector_PinHeader_2.54mm:PinHeader_1x02_P2.54mm_Vertical, F.Cu at (56.7, 84.4)
- added J2: I2, Connector_PinHeader_2.54mm:PinHeader_1x02_P2.54mm_Vertical, F.Cu at (221.8, 155.5)
- added J3: I3, Connector_PinHeader_2.54mm:PinHeader_1x02_P2.54mm_Vertical, F.Cu at (64.0, 75.0)
- added J3: I3, Connector_PinHeader_2.54mm:PinHeader_1x02_P2.54mm_Vertical, F.Cu at (64.0, 146.1)
- added J3: I3, Connector_PinHeader_2.54mm:PinHeader_1x02_P2.54mm_Vertical, F.Cu at (229.1, 146.1)
- added J3: I3, Connector_PinHeader_2.54mm:PinHeader_1x02_P2.54mm_Vertical, F.Cu at (229.1, 75.0)
- added J3: I3, Connector_PinHeader_2.54mm:PinHeader_1x02_P2.54mm_Vertical, F.Cu at (145.3, 146.1)
- added J4: gnd, Connector_PinHeader_2.54mm:PinHeader_1x01_P2.54mm_Vertical, F.Cu at (142.6, 161.8)
- added J4: gnd, Connector_PinHeader_2.54mm:PinHeader_1x01_P2.54mm_Vertical, F.Cu at (226.4, 161.8)
- added J4: gnd, Connector_PinHeader_2.54mm:PinHeader_1x01_P2.54mm_Vertical, F.Cu at (61.3, 90.7)
- added J4: gnd, Connector_PinHeader_2.54mm:PinHeader_1x01_P2.54mm_Vertical, F.Cu at (226.4, 90.7)
- added J4: gnd, Connector_PinHeader_2.54mm:PinHeader_1x01_P2.54mm_Vertical, F.Cu at (61.3, 161.8)
- added J5: out, TerminalBlock_Phoenix:TerminalBlock_Phoenix_MKDS-1,5-2-5.08_1x02_P5.08mm_Horizontal, F.Cu at (252.7, 71.8)
- added J5: out, TerminalBlock_Phoenix:TerminalBlock_Phoenix_MKDS-1,5-2-5.08_1x02_P5.08mm_Horizontal, F.Cu at (168.9, 142.9)
- added J5: out, TerminalBlock_Phoenix:TerminalBlock_Phoenix_MKDS-1,5-2-5.08_1x02_P5.08mm_Horizontal, F.Cu at (87.6, 71.8)
- added J5: out, TerminalBlock_Phoenix:TerminalBlock_Phoenix_MKDS-1,5-2-5.08_1x02_P5.08mm_Horizontal, F.Cu at (252.7, 142.9)
- added J5: out, TerminalBlock_Phoenix:TerminalBlock_Phoenix_MKDS-1,5-2-5.08_1x02_P5.08mm_Horizontal, F.Cu at (87.6, 142.9)
- added J6: V1, Connector_PinHeader_2.54mm:PinHeader_1x01_P2.54mm_Vertical, F.Cu at (197.8, 142.6)
- added J6: V1, Connector_PinHeader_2.54mm:PinHeader_1x01_P2.54mm_Vertical, F.Cu at (197.8, 71.5)
- added J6: V1, Connector_PinHeader_2.54mm:PinHeader_1x01_P2.54mm_Vertical, F.Cu at (114.0, 142.6)
- added J6: V1, Connector_PinHeader_2.54mm:PinHeader_1x01_P2.54mm_Vertical, F.Cu at (32.7, 142.6)
- added J6: V1, Connector_PinHeader_2.54mm:PinHeader_1x01_P2.54mm_Vertical, F.Cu at (32.7, 71.5)
- added J7: in, TerminalBlock_Phoenix:TerminalBlock_Phoenix_MKDS-1,5-2-5.08_1x02_P5.08mm_Horizontal, F.Cu at (51.0, 121.3)
- added J7: in, TerminalBlock_Phoenix:TerminalBlock_Phoenix_MKDS-1,5-2-5.08_1x02_P5.08mm_Horizontal, F.Cu at (51.0, 50.2)
- added J7: in, TerminalBlock_Phoenix:TerminalBlock_Phoenix_MKDS-1,5-2-5.08_1x02_P5.08mm_Horizontal, F.Cu at (216.1, 50.2)
- added J7: in, TerminalBlock_Phoenix:TerminalBlock_Phoenix_MKDS-1,5-2-5.08_1x02_P5.08mm_Horizontal, F.Cu at (216.1, 121.3)
- added J7: in, TerminalBlock_Phoenix:TerminalBlock_Phoenix_MKDS-1,5-2-5.08_1x02_P5.08mm_Horizontal, F.Cu at (132.3, 121.3)
- added Q1: BD140, Package_TO_SOT_THT:TO-126-3_Vertical, F.Cu at (43.4, 137.1)
- added Q1: BD140, Package_TO_SOT_THT:TO-126-3_Vertical, F.Cu at (208.5, 66.0)
- added Q1: BD140, Package_TO_SOT_THT:TO-126-3_Vertical, F.Cu at (208.5, 137.1)
- added Q1: BD140, Package_TO_SOT_THT:TO-126-3_Vertical, F.Cu at (43.4, 66.0)
- added Q1: BD140, Package_TO_SOT_THT:TO-126-3_Vertical, F.Cu at (124.7, 137.1)
- added Q10: BD139, Package_TO_SOT_THT:TO-126-3_Vertical, F.Cu at (44.0, 89.5)
- added Q10: BD139, Package_TO_SOT_THT:TO-126-3_Vertical, F.Cu at (44.0, 160.6)
- added Q10: BD139, Package_TO_SOT_THT:TO-126-3_Vertical, F.Cu at (125.3, 160.6)
- added Q10: BD139, Package_TO_SOT_THT:TO-126-3_Vertical, F.Cu at (209.1, 160.6)
- added Q10: BD139, Package_TO_SOT_THT:TO-126-3_Vertical, F.Cu at (209.1, 89.5)
- added Q2: BD140, Package_TO_SOT_THT:TO-126-3_Vertical, F.Cu at (224.1, 60.4)
- added Q2: BD140, Package_TO_SOT_THT:TO-126-3_Vertical, F.Cu at (59.0, 60.4)
- added Q2: BD140, Package_TO_SOT_THT:TO-126-3_Vertical, F.Cu at (224.1, 131.5)
- added Q2: BD140, Package_TO_SOT_THT:TO-126-3_Vertical, F.Cu at (140.3, 131.5)
- added Q2: BD140, Package_TO_SOT_THT:TO-126-3_Vertical, F.Cu at (59.0, 131.5)
- added Q3: BD139, Package_TO_SOT_THT:TO-126-3_Vertical, F.Cu at (130.1, 142.7)
- added Q3: BD139, Package_TO_SOT_THT:TO-126-3_Vertical, F.Cu at (48.8, 71.6)
- added Q3: BD139, Package_TO_SOT_THT:TO-126-3_Vertical, F.Cu at (48.8, 142.7)
- added Q3: BD139, Package_TO_SOT_THT:TO-126-3_Vertical, F.Cu at (213.9, 71.6)
- added Q3: BD139, Package_TO_SOT_THT:TO-126-3_Vertical, F.Cu at (213.9, 142.7)
- added Q4: BD139, Package_TO_SOT_THT:TO-126-3_Vertical, F.Cu at (219.0, 139.1)
- added Q4: BD139, Package_TO_SOT_THT:TO-126-3_Vertical, F.Cu at (135.2, 139.1)
- added Q4: BD139, Package_TO_SOT_THT:TO-126-3_Vertical, F.Cu at (53.9, 139.1)
- added Q4: BD139, Package_TO_SOT_THT:TO-126-3_Vertical, F.Cu at (53.9, 68.0)
- added Q4: BD139, Package_TO_SOT_THT:TO-126-3_Vertical, F.Cu at (219.0, 68.0)
- added Q5: TIP42C, Package_TO_SOT_THT:TO-220-3_Vertical, F.Cu at (240.0, 48.0)
- added Q5: TIP42C, Package_TO_SOT_THT:TO-220-3_Vertical, F.Cu at (74.9, 119.1)
- added Q5: TIP42C, Package_TO_SOT_THT:TO-220-3_Vertical, F.Cu at (74.9, 48.0)
- added Q5: TIP42C, Package_TO_SOT_THT:TO-220-3_Vertical, F.Cu at (156.2, 119.1)
- added Q5: TIP42C, Package_TO_SOT_THT:TO-220-3_Vertical, F.Cu at (240.0, 119.1)
- added Q6: BD139, Package_TO_SOT_THT:TO-126-3_Vertical, F.Cu at (150.1, 131.4)
- added Q6: BD139, Package_TO_SOT_THT:TO-126-3_Vertical, F.Cu at (68.8, 60.3)
- added Q6: BD139, Package_TO_SOT_THT:TO-126-3_Vertical, F.Cu at (233.9, 131.4)
- added Q6: BD139, Package_TO_SOT_THT:TO-126-3_Vertical, F.Cu at (233.9, 60.3)
- added Q6: BD139, Package_TO_SOT_THT:TO-126-3_Vertical, F.Cu at (68.8, 131.4)
- added Q7: BD139, Package_TO_SOT_THT:TO-126-3_Vertical, F.Cu at (53.9, 147.3)
- added Q7: BD139, Package_TO_SOT_THT:TO-126-3_Vertical, F.Cu at (219.0, 147.3)
- added Q7: BD139, Package_TO_SOT_THT:TO-126-3_Vertical, F.Cu at (53.9, 76.2)
- added Q7: BD139, Package_TO_SOT_THT:TO-126-3_Vertical, F.Cu at (135.2, 147.3)
- added Q7: BD139, Package_TO_SOT_THT:TO-126-3_Vertical, F.Cu at (219.0, 76.2)
- added Q8: BD139, Package_TO_SOT_THT:TO-126-3_Vertical, F.Cu at (216.2, 160.6)
- added Q8: BD139, Package_TO_SOT_THT:TO-126-3_Vertical, F.Cu at (216.2, 89.5)
- added Q8: BD139, Package_TO_SOT_THT:TO-126-3_Vertical, F.Cu at (51.1, 89.5)
- added Q8: BD139, Package_TO_SOT_THT:TO-126-3_Vertical, F.Cu at (132.3, 160.6)
- added Q8: BD139, Package_TO_SOT_THT:TO-126-3_Vertical, F.Cu at (51.1, 160.6)
- added R1: 390, Resistor_THT:R_Axial_DIN0204_L3.6mm_D1.6mm_P5.08mm_Horizontal, F.Cu at (44.0, 146.6)
- added R1: 390, Resistor_THT:R_Axial_DIN0204_L3.6mm_D1.6mm_P5.08mm_Horizontal, F.Cu at (44.0, 75.5)
- added R1: 390, Resistor_THT:R_Axial_DIN0204_L3.6mm_D1.6mm_P5.08mm_Horizontal, F.Cu at (125.3, 146.6)
- added R1: 390, Resistor_THT:R_Axial_DIN0204_L3.6mm_D1.6mm_P5.08mm_Horizontal, F.Cu at (209.1, 75.4)
- added R1: 390, Resistor_THT:R_Axial_DIN0204_L3.6mm_D1.6mm_P5.08mm_Horizontal, F.Cu at (209.1, 146.6)
- added R2: 1k, Resistor_THT:R_Axial_DIN0204_L3.6mm_D1.6mm_P5.08mm_Horizontal, F.Cu at (240.0, 144.1)
- added R2: 1k, Resistor_THT:R_Axial_DIN0204_L3.6mm_D1.6mm_P5.08mm_Horizontal, F.Cu at (74.9, 144.1)
- added R2: 1k, Resistor_THT:R_Axial_DIN0204_L3.6mm_D1.6mm_P5.08mm_Horizontal, F.Cu at (156.1, 144.1)
- added R2: 1k, Resistor_THT:R_Axial_DIN0204_L3.6mm_D1.6mm_P5.08mm_Horizontal, F.Cu at (240.0, 73.0)
- added R2: 1k, Resistor_THT:R_Axial_DIN0204_L3.6mm_D1.6mm_P5.08mm_Horizontal, F.Cu at (74.9, 73.0)
- added R3: 470, Resistor_THT:R_Axial_DIN0204_L3.6mm_D1.6mm_P5.08mm_Horizontal, F.Cu at (38.3, 137.5)
- added R3: 470, Resistor_THT:R_Axial_DIN0204_L3.6mm_D1.6mm_P5.08mm_Horizontal, F.Cu at (203.4, 137.5)
- added R3: 470, Resistor_THT:R_Axial_DIN0204_L3.6mm_D1.6mm_P5.08mm_Horizontal, F.Cu at (38.3, 66.4)
- added R3: 470, Resistor_THT:R_Axial_DIN0204_L3.6mm_D1.6mm_P5.08mm_Horizontal, F.Cu at (119.6, 137.5)
- added R3: 470, Resistor_THT:R_Axial_DIN0204_L3.6mm_D1.6mm_P5.08mm_Horizontal, F.Cu at (203.4, 66.4)
- added R4: 2, Resistor_THT:R_Axial_DIN0204_L3.6mm_D1.6mm_P5.08mm_Horizontal, F.Cu at (83.0, 56.5)
- added R4: 2, Resistor_THT:R_Axial_DIN0204_L3.6mm_D1.6mm_P5.08mm_Horizontal, F.Cu at (248.1, 56.4)
- added R4: 2, Resistor_THT:R_Axial_DIN0204_L3.6mm_D1.6mm_P5.08mm_Horizontal, F.Cu at (164.3, 127.6)
- added R4: 2, Resistor_THT:R_Axial_DIN0204_L3.6mm_D1.6mm_P5.08mm_Horizontal, F.Cu at (83.0, 127.6)
- added R4: 2, Resistor_THT:R_Axial_DIN0204_L3.6mm_D1.6mm_P5.08mm_Horizontal, F.Cu at (248.1, 127.6)
- added R5: 470, Resistor_THT:R_Axial_DIN0204_L3.6mm_D1.6mm_P5.08mm_Horizontal, F.Cu at (84.4, 80.7)
- added R5: 470, Resistor_THT:R_Axial_DIN0204_L3.6mm_D1.6mm_P5.08mm_Horizontal, F.Cu at (165.7, 151.8)
- added R5: 470, Resistor_THT:R_Axial_DIN0204_L3.6mm_D1.6mm_P5.08mm_Horizontal, F.Cu at (249.5, 151.8)
- added R5: 470, Resistor_THT:R_Axial_DIN0204_L3.6mm_D1.6mm_P5.08mm_Horizontal, F.Cu at (84.4, 151.8)
- added R5: 470, Resistor_THT:R_Axial_DIN0204_L3.6mm_D1.6mm_P5.08mm_Horizontal, F.Cu at (249.5, 80.7)
- added R6: 470, Resistor_THT:R_Axial_DIN0204_L3.6mm_D1.6mm_P5.08mm_Horizontal, F.Cu at (234.8, 152.1)
- added R6: 470, Resistor_THT:R_Axial_DIN0204_L3.6mm_D1.6mm_P5.08mm_Horizontal, F.Cu at (69.7, 152.1)
- added R6: 470, Resistor_THT:R_Axial_DIN0204_L3.6mm_D1.6mm_P5.08mm_Horizontal, F.Cu at (69.7, 81.0)
- added R6: 470, Resistor_THT:R_Axial_DIN0204_L3.6mm_D1.6mm_P5.08mm_Horizontal, F.Cu at (151.0, 152.1)
- added R6: 470, Resistor_THT:R_Axial_DIN0204_L3.6mm_D1.6mm_P5.08mm_Horizontal, F.Cu at (234.8, 81.0)
- added R7: 470, Resistor_THT:R_Axial_DIN0204_L3.6mm_D1.6mm_P5.08mm_Horizontal, F.Cu at (74.6, 56.5)
- added R7: 470, Resistor_THT:R_Axial_DIN0204_L3.6mm_D1.6mm_P5.08mm_Horizontal, F.Cu at (155.9, 127.6)
- added R7: 470, Resistor_THT:R_Axial_DIN0204_L3.6mm_D1.6mm_P5.08mm_Horizontal, F.Cu at (239.7, 56.5)
- added R7: 470, Resistor_THT:R_Axial_DIN0204_L3.6mm_D1.6mm_P5.08mm_Horizontal, F.Cu at (239.7, 127.6)
- added R7: 470, Resistor_THT:R_Axial_DIN0204_L3.6mm_D1.6mm_P5.08mm_Horizontal, F.Cu at (74.6, 127.6)
- added R8: 100, Resistor_THT:R_Axial_DIN0204_L3.6mm_D1.6mm_P5.08mm_Horizontal, F.Cu at (203.5, 61.3)
- added R8: 100, Resistor_THT:R_Axial_DIN0204_L3.6mm_D1.6mm_P5.08mm_Horizontal, F.Cu at (38.4, 132.4)
- added R8: 100, Resistor_THT:R_Axial_DIN0204_L3.6mm_D1.6mm_P5.08mm_Horizontal, F.Cu at (203.5, 132.4)
- added R8: 100, Resistor_THT:R_Axial_DIN0204_L3.6mm_D1.6mm_P5.08mm_Horizontal, F.Cu at (119.6, 132.4)
- added R8: 100, Resistor_THT:R_Axial_DIN0204_L3.6mm_D1.6mm_P5.08mm_Horizontal, F.Cu at (38.4, 61.3)
- added R9: 100, Resistor_THT:R_Axial_DIN0204_L3.6mm_D1.6mm_P5.08mm_Horizontal, F.Cu at (59.0, 47.5)
- added R9: 100, Resistor_THT:R_Axial_DIN0204_L3.6mm_D1.6mm_P5.08mm_Horizontal, F.Cu at (224.1, 118.6)
- added R9: 100, Resistor_THT:R_Axial_DIN0204_L3.6mm_D1.6mm_P5.08mm_Horizontal, F.Cu at (59.0, 118.6)
- added R9: 100, Resistor_THT:R_Axial_DIN0204_L3.6mm_D1.6mm_P5.08mm_Horizontal, F.Cu at (224.1, 47.4)
- added R9: 100, Resistor_THT:R_Axial_DIN0204_L3.6mm_D1.6mm_P5.08mm_Horizontal, F.Cu at (140.3, 118.6)
- added U1: TL431LP, Package_TO_SOT_THT:TO-92_Inline, F.Cu at (203.2, 146.8)
- added U1: TL431LP, Package_TO_SOT_THT:TO-92_Inline, F.Cu at (119.4, 146.8)
- added U1: TL431LP, Package_TO_SOT_THT:TO-92_Inline, F.Cu at (38.1, 146.8)
- added U1: TL431LP, Package_TO_SOT_THT:TO-92_Inline, F.Cu at (38.1, 75.7)
- added U1: TL431LP, Package_TO_SOT_THT:TO-92_Inline, F.Cu at (203.2, 75.7)
- C4: footprint Capacitor_THT:C_Rect_L16.5mm_W4.7mm_P15.00mm_MKT -> Capacitor_THT:C_Rect_L7.0mm_W2.0mm_P5.00mm
- moved C4 9.77 mm to (149.9, 66.7)
Routing:
- net Net-(J5-Pin_2): track 67.1 -> 402.6 mm
- net Net-(J7-Pin_2): track 58.2 -> 345.6 mm
- net Net-(Q7-B): track 57.2 -> 342.9 mm
- net Net-(Q2-C): track 35.3 -> 211.5 mm
- net Net-(J1-Pin_2): track 32.7 -> 196.0 mm
- net Net-(J6-Pin_1): track 25.7 -> 150.4 mm
- net Net-(J2-Pin_1): track 22.7 -> 136.1 mm
- net Net-(J3-Pin_1): track 17.7 -> 106.0 mm
- net Net-(Q1-B): track 16.8 -> 101.1 mm
- net Net-(Q5-B): track 16.3 -> 98.0 mm
- net Net-(J1-Pin_1): track 16.3 -> 97.8 mm
- net Net-(Q10-B): track 13.5 -> 80.8 mm
- net Net-(J3-Pin_2): track 8.22 -> 49.3 mm
- net Net-(Q2-E): track 7.85 -> 47.1 mm
- net Net-(J2-Pin_2): track 5.62 -> 33.7 mm
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Other:
- board size 64 x 51 mm -> 229.1 x 122.1 mm
